File: smd-converter.sch (KiCad schematic (older format))
At the start: 2 parts, among them J1 Conn_01x08_Male, U1 LT6234

Commit message: Add files via upload
Parts:
- J1: footprint Package_DIP:DIP-8_W7.62mm -> tastatur:DIP-8_W7.62mm-adapter
Changed lines of the file:
@@
 F 0 "J1" H 4322 2624 50  0000 R CNN
 F 1 "Conn_01x08_Male" H 4322 2533 50  0000 R CNN
-F 2 "Package_DIP:DIP-8_W7.62mm" H 4350 2650 50  0001 C CNN
+F 2 "tastatur:DIP-8_W7.62mm-adapter" H 4350 2650 50  0001 C CNN
 F 3 "~" H 4350 2650 50  0001 C CNN
 	1    4350 2650
