File: smd-converter.kicad_pcb (KiCad board)
At the start: 2 copper layers, 11.5 x 12.5 mm, 2 parts, among them J1 Conn_01x08_Male, U1 LT6234

Commit message: Add files via upload
Parts:
- J1: footprint Package_DIP:DIP-8_W7.62mm -> tastatur:DIP-8_W7.62mm-adapter
Other:
- net class Default: clearance 0.2 -> 0.13
- rule trace_clearance: 0.2 -> 0.13

Commit message: Add files via upload
Other:
- board size 11.5 x 12.5 mm -> 11.5 x 12.8 mm
Changed lines of the file:
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@@
       (effects (font (size 1 1) (thickness 0.15)))
     )
-    (fp_text value LT6234 (at -0.075 -0.115 180) (layer F.SilkS)
+    (fp_text value LT6234 (at 5.925 0.135 180) (layer F.SilkS)
       (effects (font (size 1 0.9) (thickness 0.15)))
     )
@@
     (effects (font (size 1.5 1.5) (thickness 0.3)))
   )
-  (gr_line (start 51.5 36.5) (end 51.5 24) (layer Edge.Cuts) (width 0.05))
+  (gr_line (start 51.5 36.5) (end 51.5 23.75) (layer Edge.Cuts) (width 0.05))
   (gr_line (start 63 36.5) (end 51.5 36.5) (layer Edge.Cuts) (width 0.05))
   (gr_line (start 63 36) (end 63 36.5) (layer Edge.Cuts) (width 0.05))
-  (gr_line (start 63 24) (end 63 36) (layer Edge.Cuts) (width 0.05))
-  (gr_line (start 51.5 24) (end 63 24) (layer Edge.Cuts) (width 0.05))
+  (gr_line (start 63 23.75) (end 63 36) (layer Edge.Cuts) (width 0.05))
+  (gr_line (start 51.5 23.75) (end 63 23.75) (layer Edge.Cuts) (width 0.05))
   (segment (start 56.3844 34.2049) (end 55.46 33.2805) (width 0.25) (layer F.Cu) (net 1))
   (segment (start 55.46 33.2805) (end 55.46 33) (width 0.25) (layer F.Cu) (net 1))
@@
     (polygon
       (pts
-        (xy 63 36.5) (xy 51.5 36.5) (xy 51.5 24) (xy 63 24)
+        (xy 63 36.25) (xy 51.5 36.25) (xy 51.5 23.75) (xy 63 23.75)
       )
     )
@@
     (polygon
       (pts
-        (xy 63 36.5) (xy 51.5 36.5) (xy 51.5 24) (xy 63 24)
+        (xy 63 36.5) (xy 51.5 36.5) (xy 51.5 23.75) (xy 63 23.75)
       )
     )
